File: schematics/keypad.kicad_sch (KiCad schematic)
At the start: 24 parts, among them J1 Conn_01x02, J2 I2C OLED Display, U1 RP2040, U2 W25Q128JVS, Y1 ASE-12MHz

Commit message: Added schematics
Parts:
- removed C1, C14, C15: 100n, symbol Device:C
- removed J1: Conn_01x02, symbol Connector_Generic:Conn_01x02
- removed R1: 1k, symbol Device:R
- removed U2: W25Q128JVS, Package_SO:SOIC-8_5.3x5.3mm_P1.27mm, symbol Memory_Flash:W25Q128JVS
- removed Y1: ASE-12MHz, Oscillator:Oscillator_SMD_Abracon_ASE-4Pin_3.2x2.5mm, symbol Oscillator:ASE-xxxMHz
Connections:
- net QSPI_CSN: no longer names the net of U1.56 (QSPI_SS)
- net QSPI_SCLK: no longer names the net of U1.52 (QSPI_SCLK)
- net QSPI_SIO_0: no longer names the net of U1.53 (QSPI_SD0)
- net QSPI_SIO_1: no longer names the net of U1.55 (QSPI_SD1)
- net QSPI_SIO_2: no longer names the net of U1.54 (QSPI_SD2)
- net QSPI_SIO_3: no longer names the net of U1.51 (QSPI_SD3)
- net XIN: no longer names the net of U1.20 (XIN)
- net XOUT: no longer names the net of U1.21 (XOUT)
Other:
- note removed: "Crystal"
- note removed: "Flash"
